Commit message: fix(metal_arm_driver): correct bundled URDF mesh refs to metal_arm_description + lowercase (final-review Important); doc: ROS-base prereq note

File: src/metal_arm_driver/urdf/metal_no_gripper.urdf (robot description, URDF)
Before this commit: robot metal, 8 links, 7 joints
Links:
- link Link1: geometry collision mesh filename=package://metal_arm_description/meshes/link1.STL; visual mesh filename=package://metal_arm_description/meshes/link1.STL
- link Link2: geometry collision mesh filename=package://metal_arm_description/meshes/link2.STL; visual mesh filename=package://metal_arm_description/meshes/link2.STL
- link Link3: geometry collision mesh filename=package://metal_arm_description/meshes/link3.STL; visual mesh filename=package://metal_arm_description/meshes/link3.STL
- link Link4: geometry collision mesh filename=package://metal_arm_description/meshes/link4.STL; visual mesh filename=package://metal_arm_description/meshes/link4.STL
- link Link5: geometry collision mesh filename=package://metal_arm_description/meshes/link5.STL; visual mesh filename=package://metal_arm_description/meshes/link5.STL
- link Link6: geometry collision mesh filename=package://metal_arm_description/meshes/link6.STL; visual mesh filename=package://metal_arm_description/meshes/link6.STL
- link base_link: geometry collision mesh filename=package://metal_arm_description/meshes/base_link.STL; visual mesh filename=package://metal_arm_description/meshes/base_link.STL

File: src/metal_arm_driver/urdf/metal_with_gripper.urdf (robot description, URDF)
Before this commit: robot metal, 8 links, 7 joints
Links:
- link Link1: geometry collision mesh filename=package://metal_arm_description/meshes/link1.STL; visual mesh filename=package://metal_arm_description/meshes/link1.STL
- link Link2: geometry collision mesh filename=package://metal_arm_description/meshes/link2.STL; visual mesh filename=package://metal_arm_description/meshes/link2.STL
- link Link3: geometry collision mesh filename=package://metal_arm_description/meshes/link3.STL; visual mesh filename=package://metal_arm_description/meshes/link3.STL
- link Link4: geometry collision mesh filename=package://metal_arm_description/meshes/link4.STL; visual mesh filename=package://metal_arm_description/meshes/link4.STL
- link Link5: geometry collision mesh filename=package://metal_arm_description/meshes/link5.STL; visual mesh filename=package://metal_arm_description/meshes/link5.STL
- link Link6: geometry collision mesh filename=package://metal_arm_description/meshes/link6.STL; visual mesh filename=package://metal_arm_description/meshes/link6.STL
- link base_link: geometry collision mesh filename=package://metal_arm_description/meshes/base_link.STL; visual mesh filename=package://metal_arm_description/meshes/base_link.STL
